File: spdif.kicad_sch (KiCad schematic)
At the start: 1 part

Commit message: Add decoupling transformer
Parts:
- added T1: PE-65612NL, Library:PE65612NL, symbol tda1541:PE-65612NL
Changed lines of the file:
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@@
 	(paper "A3")
+	(symbol
+		(lib_id "tda1541:PE-65612NL")
+		(at 88.9 93.98 0)
+		(unit 1)
+		(exclude_from_sim no)
+		(in_bom yes)
+		(on_board yes)
+		(dnp no)
+		(fields_autoplaced yes)
+		(property "Reference" "T1"
+			(at 99.06 86.36 0)
+			(effects
+				(font
+					(size 1.27 1.27)
+				)
+			)
+		)
+		(property "Value" "PE-65612NL"
+			(at 99.06 88.9 0)
+			(effects
+				(font
+					(size 1.27 1.27)
+				)
+			)
+		)
+		(property "Footprint" "Library:PE65612NL"
+			(at 105.41 91.44 0)
+			(effects
+				(font
+					(size 1.27 1.27)
+				)
+				(justify left)
+				(hide yes)
+			)
+		)
+		(property "Datasheet" "https://www.digikey.ph/en/products/detail/pulse-electronics/PE-65612NL/1812213?msockid=3bdc366bbe0663d83c1223c0bf3662a6"
+			(at 89.662 104.394 0)
+			(effects
+				(font
+					(size 1.27 1.27)
+				)
+				(justify left)
+				(hide yes)
+			)
+		)
+		(property "Description" "Audio Transformers / Signal Transformers THT Digital Audio 2500uH 1-Port"
+			(at 102.616 81.28 0)
+			(effects
+				(font
+					(size 1.27 1.27)
+				)
+				(hide yes)
+			)
+		)
+		(property "Description_1" "Audio Transformers / Signal Transformers THT Digital Audio 2500uH 1-Port"
+			(at 89.662 106.934 0)
+			(effects
+				(font
+					(size 1.27 1.27)
+				)
+				(justify left)
+				(hide yes)
+			)
+		)
+		(property "Height" "6.6"
+			(at 105.41 99.06 0)
+			(effects
+				(font
+					(size 1.27 1.27)
+				)
+				(justify left)
+				(hide yes)
+			)
+		)
+		(property "Manufacturer_Name" "Pulse Electronics"
+			(at 89.662 112.014 0)
+			(effects
+				(font
+					(size 1.27 1.27)
+				)
+				(justify left)
+				(hide yes)
+			)
+		)
+		(property "Manufacturer_Part_Number" "PE-65612NL"
+			(at 89.662 114.554 0)
+			(effects
+				(font
+					(size 1.27 1.27)
+				)
+				(justify left)
+				(hide yes)
+			)
+		)
+		(property "Mouser Part Number" "673-PE-65612NL"
+			(at 89.916 117.856 0)
+			(effects
+				(font
+					(size 1.27 1.27)
+				)
+				(justify left)
+				(hide yes)
+			)
+		)
+		(property "Mouser Price/Stock" "https://www.mouser.co.uk/ProductDetail/Pulse-Electronics/PE-65612NL?qs=0Ba7fqpihnjaWgPSZtGigw%3D%3D"
+			(at 89.662 119.634 0)
+			(effects
+				(font
+					(size 1.27 1.27)
+				)
+				(justify left)
+				(hide yes)
+			)
+		)
+		(property "Arrow Part Number" "PE-65612NL"
+			(at 89.662 122.174 0)
+			(effects
+				(font
+					(size 1.27 1.27)
+				)
+				(justify left)
+				(hide yes)
+			)
+		)
+		(property "Arrow Price/Stock" "https://www.arrow.com/en/products/pe-65612nl/pulse-electronics-corporation?utm_currency=USD&region=nac"
+			(at 89.662 124.714 0)
+			(effects
+				(font
+					(size 1.27 1.27)
+				)
+				(justify left)
+				(hide yes)
+			)
+		)
+		(pin "1"
+		)
+		(pin "4"
+		)
+		(pin "2"
+		)
+		(pin "3"
+		)
+		(instances
+			(project ""
+				(path "/e63e39d7-6ac0-4ffd-8aa3-1841a4541b55/d70013f8-cc00-4f06-af80-5a33e2840dec"
+					(reference "T1")
+					(unit 1)
+				)
+			)
+		)
+	)
 	(symbol
 		(lib_id "tda1541:TDA1315H")

Commit message: Progrees on spdif
Parts:
- added C38: 100n, symbol Device:C
- added C39: 2n2, symbol Device:C
- added C40, C43: C, symbol Device:C
- added C41, C42: C_Polarized, symbol Device:C_Polarized
- added D1, D2, D3, D4, D5: LED, symbol Device:LED
- added FB1: FerriteBead, symbol Device:FerriteBead
- added JP1: Jumper_2_Open, TestPoint:TestPoint_2Pads_Pitch2.54mm_Drill0.8mm, symbol Jumper:Jumper_2_Open
- added R34: 470r, symbol Device:R
- added R35, R36, R37, R38: 100r, symbol Device:R
- added R39, R40: R, symbol Device:R
Connections:
- net at U1.1 (RC_FIL): now also U1.44 (RCINT), C39.1, R34.2
- net at U1.12 (UNLOCK): now also D1.1 (K)
- net at U1.13 (FS32): now also D3.1 (K)
- net at U1.14 (FS44): now also D4.1 (K)
- net at U1.15 (FS48): now also D5.1 (K)
- net at U1.16 (CHMODE): now also D2.1 (K)
- net at U1.17 (VDDD2): now also U1.3 (VDDA), U1.42 (VDDD1), C40.1, C41.1, C43.2, FB1.2
- net at U1.19 (RESET): now also C42.2
- net at U1.2 (VREF): now also C38.1
- net GND: now reaches U1.20 (PD)
- net GND: now also C38.2, C39.2, C40.2, C41.2, C43.1, JP1.1 (A), R34.1
- net at U1.35 (SD): now also R35.1
- net at U1.36 (WS): now also R36.1
- net at U1.37 (SCK): now also R37.2
- net at U1.40 (SYSCLKO): now also R38.2
- net at U1.43 (CLKSEL): now also JP1.2 (B)
- new net: D2.2 (A), D3.2 (A), D4.2 (A), D5.2 (A), R40.1
- new net: D1.2 (A), R39.1
- new net: R39.2, R40.2
- new net SCK: R37.1
- new net SD: R35.2
- new net WS: R36.2
- new net syscko: R38.1
Other:
- moved on the sheet: T1
